Commit message: deleted:    check.md 	modified:   moria_gazebo/config/my_controllers.yaml 	modified:   moria_gazebo/launch/btu.launch.py 	modified:   moria_gazebo/launch/robot_state_publisher.launch.py 	modified:   moria_gazebo/model/moria.urdf 	new file:   moria_gazebo/urdf/moria.urdf 	modified:   moria_todos.md

File: moria_gazebo/urdf/moria.urdf (robot description, URDF)
Before this commit: robot moria, 16 links, 15 joints
Links:
- link base: geometry collision mesh filename=package://moria_gazebo/model/meshes/base_link.STL; visual mesh filename=package://moria_gazebo/model/meshes/base_link.STL
- link base_scan_b: geometry collision cylinder length=0.0315 radius=0.055; visual mesh filename=package://moria_gazebo/model/meshes/lidar.stl scale=0.001 0.001 0.001
- link base_scan_f: geometry collision cylinder length=0.0315 radius=0.055; visual mesh filename=package://moria_gazebo/model/meshes/lidar.stl scale=0.001 0.001 0.001
- link body: geometry collision mesh filename=package://moria_gazebo/model/meshes/body.STL; visual mesh filename=package://moria_gazebo/model/meshes/body.STL
- link camera: geometry collision mesh filename=package://moria_gazebo/model/meshes/camera.STL; visual mesh filename=package://moria_gazebo/model/meshes/camera.STL
- link left_wheel: geometry collision mesh filename=package://moria_gazebo/model/meshes/left_wheel.STL; visual mesh filename=package://moria_gazebo/model/meshes/left_wheel.STL
- link legs: geometry collision mesh filename=package://moria_gazebo/model/meshes/legs.STL; visual mesh filename=package://moria_gazebo/model/meshes/legs.STL
- link right_wheel: geometry collision mesh filename=package://moria_gazebo/model/meshes/right_wheel.STL; visual mesh filename=package://moria_gazebo/model/meshes/right_wheel.STL
