Commit message: Updated 'moria_gazebo' and 'moria_description' 	modified:   README.md 	new file:   check.md 	modified:   moria_description/rviz/model.rviz 	modified:   moria_description/urdf/moria.urdf.xacro 	modified:   moria_gazebo/launch/btu.launch.py 	modified:   moria_gazebo/launch/robot_state_publisher.launch.py 	modified:   moria_gazebo/launch/spawn_moria.launch.py 	new file:   moria_gazebo/model/meshes/one_piece_base.STL 	new file:   moria_gazebo/model/moria.sdf 	modified:   moria_gazebo/model/moria.urdf 	new file:   moria_gazebo/model/one_moria.urdf

File: moria_description/urdf/moria.urdf.xacro (robot description, xacro)
@@ -24,6 +24,6 @@
         </visual>
         <inertial>
-            <origin
-                xyz="-0.00044759 -0.044904 0.3116"/>
+		    <!--<origin xyz="-0.00044759 -0.044904 0.3116"/>-->
+            <origin xyz="0 0 -0.20"/>
             <mass
                 value="3.027" />

File: moria_gazebo/model/one_moria.urdf (robot description, URDF)
Before this commit: robot moria, 16 links, 15 joints
Links:
- removed link body
- removed link legs
Joints:
- removed joint body_joint
- removed joint legs_joint
- joint camera_joint: origin xyz=0.11656 0.00021246 0.40556 rpy=1.9635 0.014384 1.5807 -> xyz=-0.00081589 0.073103 0.95616 rpy=1.9635 0.014384 1.5807; parent body -> base
- joint caster_joint: origin xyz=0 0.20 -0.34 rpy=0 0 0 -> xyz=0 0.12 0.02 rpy=0 0 0
- joint imu_joint: origin xyz=0 0 -0.33 rpy=0 0 0 -> xyz=0 0 0.10 rpy=0 0 0
- joint left_wheel_joint: origin xyz=-0.13 -0.11 -0.33  rpy=-1.57 0 0 -> xyz=-0.13 -0.12 0.034  rpy=-1.57 0 0
- joint right_wheel_joint: origin xyz=0.13 -0.11 -0.33 rpy=1.57 0 0 -> xyz=0.13 -0.11659 0.034 rpy=1.57 0 0
- joint scan_joint_b: origin xyz=0 -0.18 -0.15 rpy=0 0 1.57 -> xyz=0 -0.18 0.15 rpy=0 0 1.57
- joint scan_joint_f: origin xyz=0 0.12 -0.15 rpy=0 0 -1.57 -> xyz=0 0.12 0.15 rpy=0 0 -1.57

Commit message: Started to build V2

File: moria_description/urdf/moria.urdf.xacro (robot description, xacro)
@@ -1,46 +1,227 @@
 <?xml version="1.0"?>
 <robot xmlns:xacro="http://www.ros.org/wiki/xacro" name="moria">
-    <xacro:include filename="inertial_macros.xacro"/>
-    <!--FLOOR DEFINITION - WORLD JOINT-->
-    <link name="floor">
-    </link>
-    <!-- ROBOT DEFINITIONS-->
-    <joint name="base_joint" type="fixed">
-        <parent link="floor"/>
-        <child link="base"/>
-        <origin xyz="1 0 0.4"/>
-    </joint>
-        <!--BASE DEFINITION-->
-    <link name="base">
-        <visual>
-            <origin xyz="0 0 0"/>
-            <geometry>
-                <mesh
-                    filename="package://moria_description/meshes/base_link.STL" />
-            </geometry>
-            <material name="">
-                <color rgba="0.79216 0.11961 0.93333 1"/>
-            </material>
-        </visual>
-        <inertial>
-		    <!--<origin xyz="-0.00044759 -0.044904 0.3116"/>-->
-            <origin xyz="0 0 -0.20"/>
-            <mass
-                value="3.027" />
-            <inertia
-                ixx="0.03787"
-                ixy="0.00001"
-                ixz="0.00001"
-                iyy="0.04356"
-                iyz="0.00008"
-                izz="0.04447"
-            />
-        </inertial>
-    </link>
-        <!--LEFT WHEEL DEFINITION-->
+    <!-- Footprint -->
+    <link name="base_footprint"/>
+    <!-- Base of the Robot -->
+    <joint name="base_footprint_joint" type="fixed">
+        <parent link="base_footprint"/>
+        <child link="base_link"/>
+        <origin xyz="0 0 0"/>
+    </joint>
+    <link name="base_link">
+        <visual>
+            <origin xyz="0 0 0" rpy="0 0 0"/>
+            <geometry>
+                <mesh filename="package://moria_description/meshes/base_link.STL"/>
+            </geometry>
+            <material name="blue">
+                <color rgba="0.0667 0.2431 0.4078 1"/>
+            </material>
+        </visual>
+        <collision>
+            <origin xyz="0 0 0" rpy="0 0 0"/>
+            <geometry>
+                <mesh filename="package://moria_description/meshes/base_link.STL"/>
+            </geometry>
+        </collision>
+        <inertial>
+            <origin xyz="0 0 0" rpy="0 0 0"/>
+            <mass value="4.44"/>
+            <inertia
+                ixx="0.02125" ixy="0.0" ixz="0.00001"
+                iyy="0.04177" iyz="0.0"
+                izz="0.04948" />
+        </inertial>
+    </link>
+    <!-- FRONT WHEEL -->
+    <joint name="front_base_joint" type="fixed">
+        <origin xyz="0.23 0 0" rpy="0 0 0"/>
+        <parent link="base_link"/>
+        <child link="front_base"/>
+    </joint>
+    <link name="front_base">
+        <visual>
+            <origin xyz="0 0 0" rpy="0 0 0"/>
+            <geometry>
+                <mesh filename="package://moria_description/meshes/front_base.STL"/>
+            </geometry>
+            <material name="blue">
+                <color rgba="0.0667 0.2431 0.4078 1"/>
+            </material>
+        </visual>
+        <collision>
+            <origin xyz="0 0 0" rpy="0 0 0"/>
+            <geometry>
+                <mesh filename="package://moria_description/meshes/front_base.STL"/>
+            </geometry>
+        </collision>
+        <inertial>
+            <origin xyz="0 0 0" rpy="0 0 0"/>
+            <mass value="0.003"/>
+            <inertia
+                ixx="0.0001" ixy="0.0" ixz="0.0"
+                iyy="0.0002" iyz="0.0"
+                izz="0.0001" />
+        </inertial>
+    </link>
+    <joint name="front_radial_joint" type="continuous">
+        <parent link="front_base"/>
+        <child link="front_radial"/>
+        <origin xyz="0 0 0" rpy="0 0 -1.5708"/>
+        <axis xyz="0 0 1"/>
+    </joint>
+    <link name="front_radial">
+        <visual>
+            <origin xyz="0 0 0" rpy="0 0 0"/>
+            <geometry>
+                <mesh filename="package://moria_description/meshes/front_rad.STL"/>
+            </geometry>
+            <material name="blue">
+                <color rgba="0.0667 0.2431 0.4078 1"/>
+            </material>
+        </visual>
+        <collision>
+            <origin xyz="0 0 0" rpy="0 0 0"/>
+            <geometry>
+                <mesh filename="package://moria_description/meshes/front_rad.STL"/>
+            </geometry>
+        </collision>
+        <inertial>
+            <origin xyz="0 0 0" rpy="0 0 0"/>
+            <mass value="0.01"/>
+            <inertia
+                ixx="2.54E-06" ixy="0.0" ixz="0.0"
+                iyy="2.17E-06" iyz="0.0"
+                izz="3.02E-06" />
+        </inertial>
+    </link>
+    <joint name="front_wheel_joint" type="continuous">
+        <parent link="front_radial"/>
+        <child link="front_wheel"/>
+        <origin xyz="0 -0.022 -0.035" rpy="1.5708 0 1.5708"/>
+        <axis xyz="0 0 -1"/>
+    </joint>
+    <link name="front_wheel">
+        <visual>
+            <origin xyz="0 0 0" rpy="0 0 0"/>
+            <geometry>
+                <mesh filename="package://moria_description/meshes/front_wheel.STL"/>
+            </geometry>
+            <material name="cyan">
+                <color rgba="0.3137 0.6941 0.7843 1"/>
+            </material>
+        </visual>
+        <collision>
+            <origin xyz="0 0 0" rpy="0 0 0"/>
+            <geometry>
+                <mesh filename="package://moria_description/meshes/front_wheel.STL"/>
+            </geometry>
+        </collision>
+        <inertial>
+            <origin xyz="0 0 0" rpy="0 0 0"/>
+            <mass value="0.006"/>
+            <inertia
+                ixx="4.60E-07" ixy="0.0" ixz="0.0"
+                iyy="4.60E-07" iyz="0.0"
+                izz="8.66E-07" />
+        </inertial>
+    </link>
+    <!-- RIGHT WHEEL-->
+    <joint name="right_motor_joint" type="fixed">
+        <parent link="base_link"/>
+        <child link="right_motor"/>
+        <origin xyz="0 -0.096 -0.02" rpy="0 0 0"/>
+    </joint>
+    <link name="right_motor">
+        <visual>
+            <origin xyz="0 0 0" rpy="0 0 0"/>
+            <geometry>
+                <mesh filename="package://moria_description/meshes/right_motor.STL"/>
+            </geometry>
+            <material name="blue">
+                <color rgba="0.0667 0.2431 0.4078 1"/>
+            </material>
+        </visual>
+        <collision>
+            <origin xyz="0 0 0" rpy="0 0 0"/>
+            <geometry>
+                <mesh filename="package://moria_description/meshes/right_motor.STL"/>
+            </geometry>
+        </collision>
+        <inertial>
+            <origin xyz="0 0 0" rpy="0 0 0"/>
+            <mass value="0.11"/>
+            <inertia
+                ixx="0.00003" ixy="0.0" ixz="0.0"
+                iyy="0.00005" iyz="0.0"
+                izz="0.00006" />
+        </inertial>
+    </link>
+    <joint name="right_wheel_joint" type="continuous">
+        <parent link="right_motor"/>
+        <child link="right_wheel"/>
+        <origin xyz="0 -0.076 0" rpy="-1.5708 0 0"/>
+        <axis xyz="0 0 1"/>
+    </joint>
+    <link name="right_wheel">
+        <visual>
+            <origin xyz="0 0 0" rpy="0 0 0"/>
+            <geometry>
+                <mesh filename="package://moria_description/meshes/right_wheel.STL"/>
+            </geometry>
+            <material name="cyan">
+                <color rgba="0.3137 0.6941 0.7843 1"/>
+            </material>
+        </visual>
+        <collision>
+            <origin xyz="0 0 0" rpy="0 0 0"/>
+            <geometry>
+                <mesh filename="package://moria_description/meshes/right_wheel.STL"/>
+            </geometry>
+        </collision>
+        <inertial>
+            <origin xyz="0 0 0" rpy="0 0 0"/>
+            <mass value="0.09111"/>
+            <inertia
+                ixx="0.00003" ixy="0.0" ixz="0.0"
+                iyy="0.00003" iyz="0.0"
+                izz="0.00004" />
+        </inertial>
+    </link>
+    <!-- LEFT WHEEL-->
+    <joint name="left_motor_joint" type="fixed">
+        <parent link="base_link"/>
+        <child link="left_motor"/>
+        <origin xyz="0 0.096 -0.02" rpy="0 0 0"/>
+    </joint>
+    <link name="left_motor">
+        <visual>
+            <origin xyz="0 0 0" rpy="0 0 0"/>
+            <geometry>
+                <mesh filename="package://moria_description/meshes/left_motor.STL"/>
+            </geometry>
+            <material name="blue">
+                <color rgba="0.0667 0.2431 0.4078 1"/>
+            </material>
+        </visual>
+        <collision>
+            <origin xyz="0 0 0" rpy="0 0 0"/>
+            <geometry>
+                <mesh filename="package://moria_description/meshes/left_motor.STL"/>
+            </geometry>
+        </collision>
+        <inertial>
+            <origin xyz="0 0 0" rpy="0 0 0"/>
+            <mass value="0.11"/>
+            <inertia
+                ixx="0.00003" ixy="0.0" ixz="0.0"
+                iyy="0.00005" iyz="0.0"
+                izz="0.00006" />
+        </inertial>
+    </link>
     <joint name="left_wheel_joint" type="continuous">
-        <parent link="base"/>
+        <parent link="left_motor"/>
         <child link="left_wheel"/>
-        <origin xyz="-0.13 -0.11 -0.33 " rpy="0 1.57 0"/>
+        <origin xyz="0 0.076 0" rpy="1.5708 0 0"/>
         <axis xyz="0 0 -1"/>
     </joint>
@@ -49,152 +230,87 @@
             <origin xyz="0 0 0" rpy="0 0 0"/>
             <geometry>
-                <cylinder
-                    radius="0.05"
-                    length="0.04"
-                />
-            </geometry>
-        </visual>
-        <xacro:inertial_cylinder
-            mass="0.0261"
-            length="0.04"
-            radius="0.05"
-        >
-            <origin xyz="0 0 0" rpy="0 0 0"/>
-        </xacro:inertial_cylinder>
-    </link>
-        <!--RIGHT WHEEL DEFINITION-->
-    <joint name="right_wheel_joint" type="continuous">
-        <parent link="base"/>
-        <child link="right_wheel"/>
-        <origin xyz="0.13 -0.11 -0.33" rpy="0 1.57 0"/>
-        <axis xyz="0 0 -1"/>
-    </joint>
-    <link name="right_wheel">
-        <visual>
-            <origin xyz="0 0 0" rpy="0 0 0"/>
-            <geometry>
-                <cylinder
-                    radius="0.05"
-                    length="0.04"
-                />
-            </geometry>
-        </visual>
-        <xacro:inertial_cylinder
-            mass="0.0261"
-            length="0.04"
-            radius="0.05"
-        >
-            <origin xyz="0 0 0" rpy="0 0 0"/>
-        </xacro:inertial_cylinder>
-    </link>
-            <!--CASTER WHEEL DEFINITION-->
-    <joint name="caster_joint" type="fixed">
-        <parent link="base"/>
-        <child link="caster_link"/>
-        <origin xyz="0 0.12 -0.36" rpy="0 0 0"/>
-    </joint>
-    <link name="caster_link">
-        <collision>
-            <origin xyz="0 0.001 0" rpy="0 0 0"/>
-            <geometry>
-                <box size="0.02 0.02 0.02"/>
-            </geometry>
-        </collision>
-        <inertial>
-            <origin xyz="0 0 0" />
-            <mass value="0.005" />
-            <inertia ixx="0.001" ixy="0.0" ixz="0.0"
-                    iyy="0.001" iyz="0.0"
-                    izz="0.001" />
-        </inertial>
-    </link>
-            <!-- LEGS DEFINITION-->
-    <joint name="legs_joint" type="fixed">
-        <origin
-            xyz="-0.0015188 -0.038639 -0.35111"
-            rpy="1.5708 0 0" />
-        <parent
-            link="base" />
-        <child
-            link="legs" />
-    </joint>
-    <link name="legs">
-        <inertial>
-            <origin
-                xyz="3.13579670600497E-05 0.410501245279509 2.92613595315391E-05"
-                rpy="0 0 0" />
-            <mass value="0.57830229100239" />
-            <inertia
-                ixx="0.00974131860411503"
-                ixy="-2.4628489310393E-06"
-                ixz="7.54615274060419E-08"
-                iyy="0.00435809920534734"
-                iyz="-2.95659056324959E-07"
-                izz="0.013324822888574" />
-        </inertial>
-        <visual>
-            <origin
-                xyz="0 0 0"
-                rpy="0 0 0" />
-            <geometry>
-                <mesh filename="package://moria_description/meshes/legs.STL" />
-            </geometry>
-            <material name="">
-                <color rgba="0.792156862745098 0.819607843137255 0.933333333333333 1" />
-            </material>
-        </visual>
-        <collision>
-            <origin
-                xyz="0 0 0"
-                rpy="0 0 0" />
-            <geometry>
-                <mesh filename="package://moria_description/meshes/legs.STL" />
-            </geometry>
-        </collision>
-    </link>
-            <!--BODY DEFINITION-->
-    <joint name="body_joint" type="fixed">
-        <origin
-            xyz="3.4229E-05 0.5421 0.029896"
-            rpy="3.1416 1.4922 -1.5708" />
-        <parent link="legs" />
-        <child link="body" />
+                <mesh filename="package://moria_description/meshes/left_wheel.STL"/>
+            </geometry>
+            <material name="cyan">
+                <color rgba="0.3137 0.6941 0.7843 1"/>
+            </material>
+        </visual>
+        <collision>
+            <origin xyz="0 0 0" rpy="0 0 0"/>
+            <geometry>
+                <mesh filename="package://moria_description/meshes/left_wheel.STL"/>
+            </geometry>
+        </collision>
+        <inertial>
+            <origin xyz="0 0 0" rpy="0 0 0"/>
+            <mass value="0.09111"/>
+            <inertia
+                ixx="0.00003" ixy="0.0" ixz="0.0"
+                iyy="0.00003" iyz="0.0"
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
File: moria_description/urdf/sensors.xacro (robot description, xacro)
@@ -1,63 +1,64 @@
 <?xml version="1.0"?>
-<robot xmlns:xacro="http://www.ros.org/wiki/xacro" >
-    <!--IMU SENSOR-->
-    <joint name="imu_joint" type="fixed">
-        <parent link="base"/>
-        <child link="imu"/>
-        <origin xyz="0 0 -0.33" rpy="0 0 0"/>
+<robot xmlns:xacro="http://www.ros.org/wiki/xacro">
+    <!-- LIDAR-->
+    <joint name="lidar_joint" type="fixed">
+        <parent link="leg"/>
+        <child link="lidar"/>
+        <origin xyz="0.1335 0.0005 0.0156" rpy="0 0 0"/>
     </joint>
-    <link name="imu"/>
-    <!--FRONT LIDAR SENSOR-->
-    <joint name="scan_joint_f" type="fixed">
-        <parent link="base"/>
-        <child link="base_scan_f"/>
-        <origin xyz="0 0.12 -0.15" rpy="0 0 -1.57"/>
-    </joint>
-    <link name="base_scan_f">
+    <link name="lidar">
         <visual>
             <origin xyz="0 0 0" rpy="0 0 0"/>
             <geometry>
-                <mesh filename="package://moria_description/meshes/lidar.stl" scale="0.001 0.001 0.001"/>
+                <mesh filename="package://moria_description/meshes/lidar.STL"/>
             </geometry>
+            <material name="cyan">
+                <color rgba="0.3137 0.6941 0.7843 1"/>
+            </material>
         </visual>
         <collision>
-            <origin xyz="0.015 0 -0.0065" rpy="0 0 0"/>
+            <origin xyz="0 0 0" rpy="0 0 0"/>
             <geometry>
-                <cylinder length="0.0315" radius="0.055"/>
+                <mesh filename="package://moria_description/meshes/lidar.STL"/>
             </geometry>
         </collision>
         <inertial>
-            <mass value="0.114" />
-            <origin xyz="0 0 0" />
-            <inertia ixx="0.001" ixy="0.0" ixz="0.0"
-                    iyy="0.001" iyz="0.0"
-                    izz="0.001" />
+            <origin xyz="0 0 0" rpy="0 0 0"/>
+            <mass value="1.33"/>
+            <inertia
+                ixx="0.00061" ixy="0.0" ixz="-0.00015"
+                iyy="0.00097" iyz="0.0"
+                izz="0.00110" />
         </inertial>
     </link>
-    <!--BACK LIDAR SENSOR-->
-    <joint name="scan_joint_b" type="fixed">
-        <parent link="base"/>
-        <child link="base_scan_b"/>
-        <origin xyz="0 -0.18 -0.15" rpy="0 0 1.57"/>
+    <!-- CAMERA-->
+    <joint name="camera_joint" type="fixed">
+        <parent link="body"/>
+        <child link="camera"/>
+        <origin xyz="0.0839 0.0004 0.507" rpy="0 0 0"/>
     </joint>
-    <link name="base_scan_b">
+    <link name="camera">
         <visual>
             <origin xyz="0 0 0" rpy="0 0 0"/>
             <geometry>
-                <mesh filename="package://moria_description/meshes/lidar.stl" scale="0.001 0.001 0.001"/>
+                <mesh filename="package://moria_description/meshes/camera.STL"/>
             </geometry>
+            <material name="cyan">
+                <color rgba="0.3137 0.6941 0.7843 1"/>
+            </material>
         </visual>
         <collision>
-            <origin xyz="0.015 0 -0.0065" rpy="0 0 0"/>
+            <origin xyz="0 0 0" rpy="0 0 0"/>
             <geometry>
-                <cylinder length="0.0315" radius="0.055"/>
+                <mesh filename="package://moria_description/meshes/camera.STL"/>
             </geometry>
         </collision>
         <inertial>
-            <mass value="0.114" />
-            <origin xyz="0 0 0" />
-            <inertia ixx="0.001" ixy="0.0" ixz="0.0"
-                    iyy="0.001" iyz="0.0"
-                    izz="0.001" />
+            <origin xyz="0 0 0" rpy="0 0 0"/>
+            <mass value="0.10791"/>
+            <inertia
+                ixx="0.00007" ixy="0.0" ixz="0.0"
+                iyy="0.000008" iyz="0.0"
+                izz="0.00007" />
         </inertial>
     </link>

Commit message: added Neck and Head of the robot. Preapared Left and Right arm files.

File: moria_description/urdf/moria.urdf.xacro (robot description, xacro)
@@ -313,4 +313,78 @@
         </inertial>
     </link>
+    <!-- HEAD-->
+    <joint name="neck_joint" type="revolute">
+        <parent link="body"/>
+        <child link="neck"/>
+        <origin xyz="0.0092 0.0004 0.5471" rpy="0 0 1.5708"/>
+        <axis xyz="0 0 1"/>
+        <limit
+            lower="-0.5"
+            upper="0.5"
+            effort="0"
+            velocity="0"/>
+    </joint>
+    <link name="neck">
+        <visual>
+            <origin xyz="0 0 0" rpy="0 0 0"/>
+            <geometry>
+                <mesh filename="package://moria_description/meshes/neck.STL"/>
+            </geometry>
+            <material name="cyan">
+                <color rgba="0.3137 0.6941 0.7843 1"/>
+            </material>
+        </visual>
+        <collision>
+            <origin xyz="0 0 0" rpy="0 0 0"/>
+            <geometry>
+                <mesh filename="package://moria_description/meshes/neck.STL"/>
+            </geometry>
+        </collision>
+        <inertial>
+            <origin xyz="0 0 0" rpy="0 0 0"/>
+            <mass value="0.046"/>
+            <inertia
+                ixx="0.00001" ixy="0.0" ixz="0.0"
+                iyy="0.00001" iyz="0.0"
+                izz="0.00001" />
+        </inertial>
+    </link>
+    <joint name="head_joint" type="revolute">
+        <parent link="neck"/>
+        <child link="head"/>
+        <origin xyz="0.0224 0.004 0.0403" rpy="1.5708 0 1.5708"/>
+        <axis xyz="0 0 1"/>
+        <limit
+            lower="-0.2"
+            upper="0.2"
+            effort="0"
+            velocity="0"/>
+    </joint>
+    <link name="head">
+        <visual>
+            <origin xyz="0 0 0" rpy="0 0 0"/>
+            <geometry>
+                <mesh filename="package://moria_description/meshes/head.STL"/>
+            </geometry>
+            <material name="cyan">
+                <color rgba="0.3137 0.6941 0.7843 1"/>
+            </material>
+        </visual>
+        <collision>
+            <origin xyz="0 0 0" rpy="0 0 0"/>
+            <geometry>
+                <mesh filename="package://moria_description/meshes/head.STL"/>
+            </geometry>
+        </collision>
+        <inertial>
+            <origin xyz="0 0 0" rpy="0 0 0"/>
+            <mass value="0.7694"/>
+            <inertia
+                ixx="0.0045" ixy="0.00005" ixz="0.0"
+                iyy="0.0029" iyz="0.0"
+                izz="0.0023" />
+        </inertial>
+    </link>
     <xacro:include filename="sensors.xacro"/>
+    <xacro:include filename="right_arm.xacro"/>
 </robot>
