Commit message: Added right arm and fingers

File: moria_description/urdf/check.urdf (robot description, URDF)
Before this commit: robot moria, 4 links, 3 joints
Links:
- added link body, mass 2.80832; collision mesh filename=package://moria_description/meshes/body.STL; visual mesh filename=package://moria_description/meshes/body.STL
- added link camera, mass 0.10791; collision mesh filename=package://moria_description/meshes/camera.STL; visual mesh filename=package://moria_description/meshes/camera.STL
- added link front_wheel, mass 0.006; collision mesh filename=package://moria_description/meshes/front_wheel.STL; visual mesh filename=package://moria_description/meshes/front_wheel.STL
- added link head, mass 0.7694; collision mesh filename=package://moria_description/meshes/head.STL; visual mesh filename=package://moria_description/meshes/head.STL
- added link left_motor, mass 0.11; collision mesh filename=package://moria_description/meshes/left_motor.STL; visual mesh filename=package://moria_description/meshes/left_motor.STL
- added link left_wheel, mass 0.09111; collision mesh filename=package://moria_description/meshes/left_wheel.STL; visual mesh filename=package://moria_description/meshes/left_wheel.STL
- added link leg, mass 2.366; collision mesh filename=package://moria_description/meshes/leg.STL; visual mesh filename=package://moria_description/meshes/leg.STL
- added link lidar, mass 1.33; collision mesh filename=package://moria_description/meshes/lidar.STL; visual mesh filename=package://moria_description/meshes/lidar.STL
- added link neck, mass 0.046; collision mesh filename=package://moria_description/meshes/neck.STL; visual mesh filename=package://moria_description/meshes/neck.STL
- added link right_motor, mass 0.11; collision mesh filename=package://moria_description/meshes/right_motor.STL; visual mesh filename=package://moria_description/meshes/right_motor.STL
- added link right_shoulder_rad, mass 0.1128; collision mesh filename=package://moria_description/meshes/right_shoulder_rad.STL; visual mesh filename=package://moria_description/meshes/right_shoulder_rad.STL
- added link right_wheel, mass 0.09111; collision mesh filename=package://moria_description/meshes/right_wheel.STL; visual mesh filename=package://moria_description/meshes/right_wheel.STL
Joints:
- added joint body_link: type fixed, parent leg, child body, origin xyz=0 0 0.465 rpy=0 0 0
- added joint camera_joint: type fixed, parent body, child camera, origin xyz=0.0839 0.0004 0.507 rpy=0 0 0
- added joint front_wheel_joint: type continuous, parent front_radial, child front_wheel, origin xyz=0 -0.022 -0.035 rpy=1.5708 0 1.5708, axis 0 0 -1
- added joint head_joint: type revolute, parent neck, child head, origin xyz=0.0224 0.004 0.0403 rpy=1.5708 0 1.5708, axis 0 0 1, limit lower=-0.2 upper=0.2 effort=0 velocity=0
- added joint left_motor_joint: type fixed, parent base_link, child left_motor, origin xyz=0 0.096 -0.02 rpy=0 0 0
- added joint left_wheel_joint: type continuous, parent left_motor, child left_wheel, origin xyz=0 0.076 0 rpy=1.5708 0 0, axis 0 0 -1
- added joint leg_joint: type fixed, parent base_link, child leg, origin xyz=0.076 0 0.185 rpy=0 0 0
- added joint lidar_joint: type fixed, parent leg, child lidar, origin xyz=0.1335 0.0005 0.0156 rpy=0 0 0
- added joint neck_joint: type revolute, parent body, child neck, origin xyz=0.0092 0.0004 0.5471 rpy=0 0 1.5708, axis 0 0 1, limit lower=-0.5 upper=0.5 effort=0 velocity=0
- added joint right_motor_joint: type fixed, parent base_link, child right_motor, origin xyz=0 -0.096 -0.02 rpy=0 0 0
- added joint right_shoulder_rad_joint: type continuous, parent body, child right_shoulder_rad, origin xyz=0 -0.1556 0.505 rpy=-1.5708 0 0, axis 0 0 1
- added joint right_wheel_joint: type continuous, parent right_motor, child right_wheel, origin xyz=0 -0.076 0 rpy=-1.5708 0 0, axis 0 0 1
- joint front_radial_joint: origin xyz=0 0 0 rpy=0 0 1.57 -> xyz=0 0 0 rpy=0 0 -1.5708

File: moria_description/urdf/right_arm.xacro (robot description, xacro)
@@ -2,9 +2,717 @@
 <robot xmlns:xacro="http://www.ros.org/wiki/xacro">
     <!-- RIGHT ARM-->
-    <!-- RIGHT HAND-->
+    <joint name="right_shoulder_rad_joint" type="continuous">
+        <parent link="body"/>
+        <child link="right_shoulder_rad"/>
+        <origin xyz="0 -0.1556 0.505" rpy="-1.5708 0 3.1416"/>
+        <axis xyz="0 0 1"/>
+    </joint>
+    <link name="right_shoulder_rad">
+        <visual>
+            <origin xyz="0 0 0" rpy="0 0 0"/>
+            <geometry>
+                <mesh
+                    filename="package://moria_description/meshes/right_shoulder_rad.STL"/>
+            </geometry>
+            <material name="blue">
+                <color rgba="0.0667 0.2431 0.4078 1"/>
+            </material>
+        </visual>
+        <collision>
+            <origin xyz="0 0 0" rpy="0 0 0"/>
+            <geometry>
+                <mesh filename="package://moria_description/meshes/right_shoulder_rad.STL"/>
+            </geometry>
+        </collision>
+        <inertial>
+            <origin xyz="0 0 0" rpy="0 0 0"/>
+            <mass value="0.1128"/>
+            <inertia
+                ixx="0.00007" ixy="0.0" ixz="0.0"
+                iyy="0.00006" iyz="0.0"
+                izz="0.00004"/>
+        </inertial>
+    </link>
+    <joint name="right_shoulder_joint" type="revolute">
+        <parent link="right_shoulder_rad"/>
+        <child link="right_shoulder"/>
+        <origin xyz="0.0258 0 0.0575" rpy="0 1.5708 0"/>
+        <axis xyz="0 0 1"/>
+        <limit
+            lower="0"
+            upper="2.5"
+            effort="0"
+            velocity="0"/>
+    </joint>
+    <link name="right_shoulder">
+        <visual>
+            <origin xyz="0 0 0" rpy="0 0 0"/>
+            <geometry>
+                <mesh filename="package://moria_description/meshes/right_shoulder.STL"/>
+            </geometry>
+            <material name="cyan">
+                <color rgba="0.3137 0.6941 0.7843 1"/>
+            </material>
+        </visual>
+        <collision>
+            <origin xyz="0 0 0" rpy="0 0 0"/>
+            <geometry>
+                <mesh filename="package://moria_description/meshes/right_shoulder.STL"/>
+            </geometry>
+        </collision>
+        <inertial>
+            <origin xyz="0 0 0" rpy="0 0 0"/>
+            <mass value="0.1576"/>
+            <inertia
+                ixx="0.00010" ixy="0.0" ixz="0.0"
+                iyy="0.00007" iyz="0.0"
+                izz="0.00011" />
+        </inertial>
+    </link>
+    <!-- UPPER ARM-->
+    <joint name="right_upper_arm_joint" type="continuous">
+        <parent link="right_shoulder"/>
+        <child link="right_upper_arm"/>
+        <origin xyz="0 0.0875 -0.0255" rpy="-1.5708 0 0"/>
+        <axis xyz="0 0 1"/>
+    </joint>
+    <link name="right_upper_arm">
+        <visual>
+            <origin xyz="0 0 0" rpy="0 0 0"/>
+            <geometry>
+                <mesh filename="package://moria_description/meshes/right_upper_arm.STL"/>
+            </geometry>
+            <material name="blue">
+                <color rgba="0.0667 0.2431 0.4078 1"/>
+            </material>
+        </visual>
+        <collision>
+            <origin xyz="0 0 0" rpy="0 0 0"/>
+            <geometry>
+                <mesh filename="package://moria_description/meshes/right_upper_arm.STL"/>
+            </geometry>
+        </collision>
+        <inertial>
+            <origin xyz="0 0 0" rpy="0 0 0"/>
+            <mass value="0.1608"/>
+            <inertia
+                ixx="0.00021" ixy="0.0" ixz="0.0"
+                iyy="0.00023" iyz="0.0"
+                izz="0.00005" />
+        </inertial>
+    </link>
+    <!-- RIGHT ELBOW-->
+    <joint name="right_elbow_joint" type="revolute">
+        <parent link="right_upper_arm"/>
+        <child link="right_elbow"/>
+        <origin xyz="-0.0226 0 0.1412" rpy="1.5708 0 -1.5708"/>
+        <axis xyz="0 0 1"/>
+        <limit
+            lower="0"
+            upper="1.5"
+            effort="0"
+            velocity="0"/>
+    </joint>
+    <link name="right_elbow">
+        <visual>
+            <origin xyz="0 0 0" rpy="0 0 0"/>
+            <geometry>
+                <mesh filename="package://moria_description/meshes/right_elbow.STL"/>
+            </geometry>
+            <material name="cyan">
+                <color rgba="0.3137 0.6941 0.7843 1"/>
+            </material>
+        </visual>
+        <collision>
+            <origin xyz="0 0 0" rpy="0 0 0"/>
+            <geometry>
+                <mesh filename="package://moria_description/meshes/right_elbow.STL"/>
+            </geometry>
+        </collision>
+        <inertial>
+            <origin xyz="0 0 0" rpy="0 0 0"/>
+            <mass value="0.1267"/>
+            <inertia
+                ixx="0.00010" ixy="0.0" ixz="0.0"
+                iyy="0.00005" iyz="0.0"
+                izz="0.00008"/>
+        </inertial>
+    </link>
+    <!-- RIGHT LOWER ARM-->
+    <joint name="right_lower_arm_joint" type="continuous">
+        <parent link="right_elbow"/>
+        <child link="right_lower_arm"/>
+        <origin xyz="0 0.0866 -0.0222" rpy="-1.5708 1.5708 0"/>
+        <axis xyz="0 0 1"/>
+    </joint>
+    <link name="right_lower_arm">
+        <visual>
+            <origin xyz="0 0 0" rpy="0 0 0"/>
+            <geometry>
+                <mesh filename="package://moria_description/meshes/right_lower_arm.STL"/>
+            </geometry>
+            <material name="blue">
+                <color rgba="0.0667 0.2431 0.4078 1"/>
+            </material>
+        </visual>
+        <collision>
+            <origin xyz="0 0 0" rpy="0 0 0"/>
+            <geometry>
+                <mesh filename="package://moria_description/meshes/right_lower_arm.STL"/>
+            </geometry>
+        </collision>
+        <inertial>
+            <origin xyz="0 0 0" rpy="0 0 0"/>
+            <mass value="0.3515"/>
+            <inertia
+                ixx="0.00033" ixy="0.0" ixz="0.0"
+                iyy="0.00033" iyz="0.0"
+                izz="0.00013" />
+        </inertial>
+    </link>
     <!-- RIGHT THUMB-->
-    <!-- RIGHT INDEX-->
-    <!-- RIGHT MIDDLE-->
-    <!-- RIGHT RING-->
+    <joint name="right_00_joint" type="revolute">
+        <parent link="right_lower_arm"/>
+        <child link="right_00"/>
+        <origin xyz="0.0063 0.0288 0.1857" rpy="2.7488 -0.0103 0.0043"/>
+        <axis xyz="0 0 1"/>
+        <limit
+            lower="0"
+            upper="1.57"
+            effort="0"
+            velocity="0"/>
+    </joint>
+    <link name="right_00">
+        <visual>
+            <origin xyz="0 0 0" rpy="0 0 0"/>
+            <geometry>
+                <mesh filename="package://moria_description/meshes/right_00.STL"/>
+            </geometry>
+            <material name="cyan">
+                <color rgba="0.3137 0.6941 0.7843 1"/>
+            </material>
+        </visual>
+        <collision>
+            <origin xyz="0 0 0" rpy="0 0 0"/>
+            <geometry>
+                <mesh filename="package://moria_description/meshes/right_00.STL"/>
+            </geometry>
+        </collision>
+        <inertial>
+            <origin xyz="0 0 0" rpy="0 0 0"/>
+            <mass value="0.005"/>
+            <inertia
+                ixx="3E-07" ixy="0.0" ixz="0.0"
+                iyy="2E-07" iyz="0.0"
+                izz="2E-07" />
+        </inertial>
+    </link>
+    <joint name="right_01_joint" type="revolute">
+        <parent link="right_00"/>
+        <child link="right_01"/>
+        <origin xyz="-0.0005 -0.0254 -0.0026" rpy="0.5632 0.9741 0.4849"/>
+        <axis xyz="0 0 1"/>
+        <limit
+            lower="0"
+            upper="1.57"
+            effort="0"
+            velocity="0"/>
+    </joint>
+    <link name="right_01">
+        <visual>
+            <origin xyz="0 0 0" rpy="0 0 0"/>
+            <geometry>
+                <mesh filename="package://moria_description/meshes/right_01.STL"/>
+            </geometry>
+            <material name="cyan">
+                <color rgba="0.3137 0.6941 0.7843 1"/>
+            </material>
+        </visual>
+        <collision>
+            <origin xyz="0 0 0" rpy="0 0 0"/>
+            <geometry>
+                <mesh filename="package://moria_description/meshes/right_01.STL"/>
+            </geometry>
+        </collision>
+        <inertial>
+            <origin xyz="0 0 0" rpy="0 0 0"/>
+            <mass value="0.002"/>
+            <inertia
+                ixx="1E-07" ixy="0.0" ixz="0.0"
+                iyy="1E-07" iyz="0.0"
+                izz="8E-08" />
+        </inertial>
+    </link>
+    <joint name="right_02_joint" type="revolute">
+        <parent link="right_01"/>
+        <child link="right_02"/>
+        <origin xyz="0.0048 -0.0246 0" rpy="0 0 0.176"/>
+        <axis xyz="0 0 1"/>
+        <limit
+            lower="0"
+            upper="1.57"
+            effort="0"
+            velocity="0"/>
+    </joint>
+    <link name="right_02">
+        <visual>
+            <origin xyz="0 0 0" rpy="0 0 0"/>
+            <geometry>
+                <mesh filename="package://moria_description/meshes/right_02.STL"/>
+            </geometry>
+            <material name="cyan">
+                <color rgba="0.3137 0.6941 0.7843 1"/>
+            </material>
+        </visual>
+        <collision>
+            <origin xyz="0 0 0" rpy="0 0 0"/>
+            <geometry>
+                <mesh filename="package://moria_description/meshes/right_02.STL"/>
+            </geometry>
+        </collision>
+        <inertial>
+            <origin xyz="0 0 0" rpy="0 0 0"/>
+            <mass value="0.002"/>
+            <inertia
+                ixx="6E-08" ixy="0.0" ixz="0.0"
+                iyy="6E-08" iyz="0.0"
+                izz="7E-08" />
+        </inertial>
+    </link>
+    <!--RIGHT INDEX-->
+    <joint name="right_10_joint" type="revolute">
+        <parent link="right_lower_arm"/>
+        <child link="right_10"/>
+        <origin xyz="0.0063 0.0269 0.2457" rpy="-1.5708 0 0.0290"/>
+        <axis xyz="0 0 1"/>
+        <limit
+            lower="0"
+            upper="1.57"
+            effort="0"
+            velocity="0"/>
+    </joint>
+    <link name="right_10">
+        <visual>
+            <origin xyz="0 0 0" rpy="0 0 0"/>
+            <geometry>
+                <mesh filename="package://moria_description/meshes/right_10.STL"/>
+            </geometry>
+            <material name="cyan">
+                <color rgba="0.3137 0.6941 0.7843 1"/>
+            </material>
+        </visual>
+        <collision>
+            <origin xyz="0 0 0" rpy="0 0 0"/>
+            <geometry>
+                <mesh filename="package://moria_description/meshes/right_10.STL"/>
+            </geometry>
+        </collision>
+        <inertial>
+            <origin xyz="0 0 0" rpy="0 0 0"/>
+            <mass value="0.002"/>
+            <inertia
+                ixx="8E-08" ixy="0.0" ixz="0.0"
+                iyy="6E-08" iyz="0.0"
+                izz="6E-08" />
+        </inertial>
+    </link>
+    <joint name="right_11_joint" type="revolute">
+        <parent link="right_10"/>
+        <child link="right_11"/>
+        <origin xyz="0 -0.024 0" rpy="0 0 0"/>
+        <axis xyz="0 0 1"/>
+        <limit
+            lower="0"
+            upper="1.57"
+            effort="0"
+            velocity="0"/>
+    </joint>
+    <link name="right_11">
+        <visual>
+            <origin xyz="0 0 0" rpy="0 0 0"/>
+            <geometry>
+                <mesh filename="package://moria_description/meshes/right_11.STL"/>
+            </geometry>
+            <material name="cyan">
+                <color rgba="0.3137 0.6941 0.7843 1"/>
+            </material>
+        </visual>
+        <collision>
+            <origin xyz="0 0 0" rpy="0 0 0"/>
+            <geometry>
+                <mesh filename="package://moria_description/meshes/right_11.STL"/>
+            </geometry>
+        </collision>
+        <inertial>
+            <origin xyz="0 0 0" rpy="0 0 0"/>
+            <mass value="0.002"/>
+            <inertia
+                ixx="6E-08" ixy="0.0" ixz="0.0"
+                iyy="5E-08" iyz="0.0"
+                izz="6E-08" />
+        </inertial>
+    </link>
+    <joint name="right_12_joint" type="revolute">
+        <parent link="right_11"/>
+        <child link="right_12"/>
+        <origin xyz="0 -0.0210 0" rpy="0 0 0"/>
+        <axis xyz="0 0 1"/>
+        <limit
+            lower="0"
+            upper="1.57"
+            effort="0"
+            velocity="0"/>
+    </joint>
+    <link name="right_12">
+        <visual>
+            <origin xyz="0 0 0" rpy="0 0 0"/>
+            <geometry>
+                <mesh filename="package://moria_description/meshes/right_12.STL"/>
+            </geometry>
+            <material name="cyan">
+                <color rgba="0.3137 0.6941 0.7843 1"/>
+            </material>
+        </visual>
+        <collision>
+            <origin xyz="0 0 0" rpy="0 0 0"/>
+            <geometry>
+                <mesh filename="package://moria_description/meshes/right_12.STL"/>
+            </geometry>
+        </collision>
+        <inertial>
+            <origin xyz="0 0 0" rpy="0 0 0"/>
+            <mass value="0.002"/>
+            <inertia
+                ixx="4E-08" ixy="0.0" ixz="0.0"
+                iyy="3E-08" iyz="0.0"
+                izz="4E-08" />
+        </inertial>
+    </link>
+    <!--RIGHT MIDDLE-->
+    <joint name="right_20_joint" type="revolute">
+        <parent link="right_lower_arm"/>
+        <child link="right_20"/>
+        <origin xyz="0.0067 0.0095 0.2457" rpy="-1.5708 0 0.0290"/>
+        <axis xyz="0 0 1"/>
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