Commit message: Added left arm, left fingers and camera's depth and rgb frames

File: moria_description/urdf/left_arm.xacro (robot description, xacro)
@@ -2,9 +2,717 @@
 <robot xmlns:xacro="http://www.ros.org/wiki/xacro">
     <!-- LEFT ARM-->
-    <!-- LEFT HAND-->
+    <joint name="left_shoulder_rad_joint" type="continuous">
+        <parent link="body"/>
+        <child link="left_shoulder_rad"/>
+        <origin xyz="0 0.1564 0.505" rpy="1.5708 0 -3.1416"/>
+        <axis xyz="0 0 -1"/>
+    </joint>
+    <link name="left_shoulder_rad">
+        <visual>
+            <origin xyz="0 0 0" rpy="0 0 0"/>
+            <geometry>
+                <mesh
+                    filename="package://moria_description/meshes/left_shoulder_rad.STL"/>
+            </geometry>
+            <material name="blue">
+                <color rgba="0.0667 0.2431 0.4078 1"/>
+            </material>
+        </visual>
+        <collision>
+            <origin xyz="0 0 0" rpy="0 0 0"/>
+            <geometry>
+                <mesh filename="package://moria_description/meshes/left_shoulder_rad.STL"/>
+            </geometry>
+        </collision>
+        <inertial>
+            <origin xyz="0 0 0" rpy="0 0 0"/>
+            <mass value="0.1109"/>
+            <inertia
+                ixx="0.00007" ixy="0.0" ixz="0.0"
+                iyy="0.00006" iyz="0.0"
+                izz="0.00004"/>
+        </inertial>
+    </link>
+    <joint name="left_shoulder_joint" type="revolute">
+        <parent link="left_shoulder_rad"/>
+        <child link="left_shoulder"/>
+        <origin xyz="0.0255 0.004 0.0575" rpy="3.14 -1.5708 0"/>
+        <axis xyz="0 0 -1"/>
+        <limit
+            lower="0"
+            upper="2.5"
+            effort="0"
+            velocity="0"/>
+    </joint>
+    <link name="left_shoulder">
+        <visual>
+            <origin xyz="0 0 0" rpy="0 0 0"/>
+            <geometry>
+                <mesh filename="package://moria_description/meshes/left_shoulder.STL"/>
+            </geometry>
+            <material name="cyan">
+                <color rgba="0.3137 0.6941 0.7843 1"/>
+            </material>
+        </visual>
+        <collision>
+            <origin xyz="0 0 0" rpy="0 0 0"/>
+            <geometry>
+                <mesh filename="package://moria_description/meshes/left_shoulder.STL"/>
+            </geometry>
+        </collision>
+        <inertial>
+            <origin xyz="0 0 0" rpy="0 0 0"/>
+            <mass value="0.1576"/>
+            <inertia
+                ixx="0.00010" ixy="0.0" ixz="0.0"
+                iyy="0.00007" iyz="0.0"
+                izz="0.00011" />
+        </inertial>
+    </link>
+    <!-- UPPER ARM-->
+    <joint name="left_upper_arm_joint" type="continuous">
+        <parent link="left_shoulder"/>
+        <child link="left_upper_arm"/>
+        <origin xyz="0 0.0875 -0.0255" rpy="-1.5708 3.14 0"/>
+        <axis xyz="0 0 -1"/>
+    </joint>
+    <link name="left_upper_arm">
+        <visual>
+            <origin xyz="0 0 0" rpy="0 0 0"/>
+            <geometry>
+                <mesh filename="package://moria_description/meshes/left_upper_arm.STL"/>
+            </geometry>
+            <material name="blue">
+                <color rgba="0.0667 0.2431 0.4078 1"/>
+            </material>
+        </visual>
+        <collision>
+            <origin xyz="0 0 0" rpy="0 0 0"/>
+            <geometry>
+                <mesh filename="package://moria_description/meshes/left_upper_arm.STL"/>
+            </geometry>
+        </collision>
+        <inertial>
+            <origin xyz="0 0 0" rpy="0 0 0"/>
+            <mass value="0.1608"/>
+            <inertia
+                ixx="0.00021" ixy="0.0" ixz="0.0"
+                iyy="0.00023" iyz="0.0"
+                izz="0.00005" />
+        </inertial>
+    </link>
+    <!-- LEFT ELBOW-->
+    <joint name="left_elbow_joint" type="revolute">
+        <parent link="left_upper_arm"/>
+        <child link="left_elbow"/>
+        <origin xyz="0.023 0 0.1412" rpy="1.5708 0 1.5708"/>
+        <axis xyz="0 0 1"/>
+        <limit
+            lower="0"
+            upper="1.5"
+            effort="0"
+            velocity="0"/>
+    </joint>
+    <link name="left_elbow">
+        <visual>
+            <origin xyz="0 0 0.425" rpy="0 0 0"/>
+            <geometry>
+                <mesh filename="package://moria_description/meshes/left_elbow.STL"/>
+            </geometry>
+            <material name="cyan">
+                <color rgba="0.3137 0.6941 0.7843 1"/>
+            </material>
+        </visual>
+        <collision>
+            <origin xyz="0 0 0" rpy="0 0 0"/>
+            <geometry>
+                <mesh filename="package://moria_description/meshes/left_elbow.STL"/>
+            </geometry>
+        </collision>
+        <inertial>
+            <origin xyz="0 0 0" rpy="0 0 0"/>
+            <mass value="0.1267"/>
+            <inertia
+                ixx="0.00010" ixy="0.0" ixz="0.0"
+                iyy="0.00005" iyz="0.0"
+                izz="0.00008"/>
+        </inertial>
+    </link>
+    <!-- LEFT LOWER ARM-->
+    <joint name="left_lower_arm_joint" type="continuous">
+        <parent link="left_elbow"/>
+        <child link="left_lower_arm"/>
+        <origin xyz="0 0.0866 -0.0234" rpy="-1.5708 2.62 0"/>
+        <axis xyz="0 0 -1"/>
+    </joint>
+    <link name="left_lower_arm">
+        <visual>
+            <origin xyz="0 0 0" rpy="0 0 0"/>
+            <geometry>
+                <mesh filename="package://moria_description/meshes/left_lower_arm.STL"/>
+            </geometry>
+            <material name="blue">
+                <color rgba="0.0667 0.2431 0.4078 1"/>
+            </material>
+        </visual>
+        <collision>
+            <origin xyz="0 0 0" rpy="0 0 0"/>
+            <geometry>
+                <mesh filename="package://moria_description/meshes/left_lower_arm.STL"/>
+            </geometry>
+        </collision>
+        <inertial>
+            <origin xyz="0 0 0" rpy="0 0 0"/>
+            <mass value="0.3515"/>
+            <inertia
+                ixx="0.00033" ixy="0.0" ixz="0.0"
+                iyy="0.00033" iyz="0.0"
+                izz="0.00013" />
+        </inertial>
+    </link>
     <!-- LEFT THUMB-->
-    <!-- LEFT INDEX-->
-    <!-- LEFT MIDDLE-->
-    <!-- LEFT RING-->
+    <joint name="left_00_joint" type="revolute">
+        <parent link="left_lower_arm"/>
+        <child link="left_00"/>
+        <origin xyz="0.0211 0.0206 0.1878" rpy="2.8403 0.2562 -0.0785"/>
+        <axis xyz="0 0 1"/>
+        <limit
+            lower="0"
+            upper="1.57"
+            effort="0"
+            velocity="0"/>
+    </joint>
+    <link name="left_00">
+        <visual>
+            <origin xyz="0 0 0" rpy="0 0 0"/>
+            <geometry>
+                <mesh filename="package://moria_description/meshes/left_00.STL"/>
+            </geometry>
+            <material name="cyan">
+                <color rgba="0.3137 0.6941 0.7843 1"/>
+            </material>
+        </visual>
+        <collision>
+            <origin xyz="0 0 0" rpy="0 0 0"/>
+            <geometry>
+                <mesh filename="package://moria_description/meshes/left_00.STL"/>
+            </geometry>
+        </collision>
+        <inertial>
+            <origin xyz="0 0 0" rpy="0 0 0"/>
+            <mass value="0.005"/>
+            <inertia
+                ixx="3E-07" ixy="0.0" ixz="0.0"
+                iyy="2E-07" iyz="0.0"
+                izz="2E-07" />
+        </inertial>
+    </link>
+    <joint name="left_01_joint" type="revolute">
+        <parent link="left_00"/>
+        <child link="left_01"/>
+        <origin xyz="0.0187 -0.0123 -0.0039" rpy="1.0739 0.0791 -0.3777"/>
+        <axis xyz="0 0 1"/>
+        <limit
+            lower="0"
+            upper="1.57"
+            effort="0"
+            velocity="0"/>
+    </joint>
+    <link name="left_01">
+        <visual>
+            <origin xyz="0 0 0" rpy="0 0 0"/>
+            <geometry>
+                <mesh filename="package://moria_description/meshes/left_01.STL"/>
+            </geometry>
+            <material name="cyan">
+                <color rgba="0.3137 0.6941 0.7843 1"/>
+            </material>
+        </visual>
+        <collision>
+            <origin xyz="0 0 0" rpy="0 0 0"/>
+            <geometry>
+                <mesh filename="package://moria_description/meshes/left_01.STL"/>
+            </geometry>
+        </collision>
+        <inertial>
+            <origin xyz="0 0 0" rpy="0 0 0"/>
+            <mass value="0.002"/>
+            <inertia
+                ixx="1E-07" ixy="0.0" ixz="0.0"
+                iyy="1E-07" iyz="0.0"
+                izz="8E-08" />
+        </inertial>
+    </link>
+    <joint name="left_02_joint" type="revolute">
+        <parent link="left_01"/>
+        <child link="left_02"/>
+        <origin xyz="0.0240 -0.0072 0" rpy="-0.2710 0.0990 0.0951"/>
+        <axis xyz="0 0 1"/>
+        <limit
+            lower="0"
+            upper="1.57"
+            effort="0"
+            velocity="0"/>
+    </joint>
+    <link name="left_02">
+        <visual>
+            <origin xyz="0 0 0" rpy="0 0 0"/>
+            <geometry>
+                <mesh filename="package://moria_description/meshes/left_02.STL"/>
+            </geometry>
+            <material name="cyan">
+                <color rgba="0.3137 0.6941 0.7843 1"/>
+            </material>
+        </visual>
+        <collision>
+            <origin xyz="0 0 0" rpy="0 0 0"/>
+            <geometry>
+                <mesh filename="package://moria_description/meshes/left_02.STL"/>
+            </geometry>
+        </collision>
+        <inertial>
+            <origin xyz="0 0 0" rpy="0 0 0"/>
+            <mass value="0.002"/>
+            <inertia
+                ixx="6E-08" ixy="0.0" ixz="0.0"
+                iyy="6E-08" iyz="0.0"
+                izz="7E-08" />
+        </inertial>
+    </link>
+    <!--LEFT INDEX-->
+    <joint name="left_10_joint" type="revolute">
+        <parent link="left_lower_arm"/>
+        <child link="left_10"/>
+        <origin xyz="0.0192 0.0186 0.2457" rpy="-1.5708 0 -0.7626"/>
+        <axis xyz="0 0 -1"/>
+        <limit
+            lower="0"
+            upper="1.57"
+            effort="0"
+            velocity="0"/>
+    </joint>
+    <link name="left_10">
+        <visual>
+            <origin xyz="0 0 0" rpy="0 0 0"/>
+            <geometry>
+                <mesh filename="package://moria_description/meshes/left_10.STL"/>
+            </geometry>
+            <material name="cyan">
+                <color rgba="0.3137 0.6941 0.7843 1"/>
+            </material>
+        </visual>
+        <collision>
+            <origin xyz="0 0 0" rpy="0 0 0"/>
+            <geometry>
+                <mesh filename="package://moria_description/meshes/left_10.STL"/>
+            </geometry>
+        </collision>
+        <inertial>
+            <origin xyz="0 0 0" rpy="0 0 0"/>
+            <mass value="0.002"/>
+            <inertia
+                ixx="8E-08" ixy="0.0" ixz="0.0"
+                iyy="6E-08" iyz="0.0"
+                izz="6E-08" />
+        </inertial>
+    </link>
+    <joint name="left_11_joint" type="revolute">
+        <parent link="left_10"/>
+        <child link="left_11"/>
+        <origin xyz="0.0010 -0.0240 0" rpy="0 0 0"/>
+        <axis xyz="0 0 -1"/>
+        <limit
+            lower="0"
+            upper="1.57"
+            effort="0"
+            velocity="0"/>
+    </joint>
+    <link name="left_11">
+        <visual>
+            <origin xyz="0 0 0" rpy="0 0 0"/>
+            <geometry>
+                <mesh filename="package://moria_description/meshes/left_11.STL"/>
+            </geometry>
+            <material name="cyan">
+                <color rgba="0.3137 0.6941 0.7843 1"/>
+            </material>
+        </visual>
+        <collision>
+            <origin xyz="0 0 0" rpy="0 0 0"/>
+            <geometry>
+                <mesh filename="package://moria_description/meshes/left_11.STL"/>
+            </geometry>
+        </collision>
+        <inertial>
+            <origin xyz="0 0 0" rpy="0 0 0"/>
+            <mass value="0.002"/>
+            <inertia
+                ixx="6E-08" ixy="0.0" ixz="0.0"
+                iyy="5E-08" iyz="0.0"
+                izz="6E-08" />
+        </inertial>
+    </link>
+    <joint name="left_12_joint" type="revolute">
+        <parent link="left_11"/>
+        <child link="left_12"/>
+        <origin xyz="0.0009 -0.0210 0" rpy="0 0 0"/>
+        <axis xyz="0 0 -1"/>
+        <limit
+            lower="0"
+            upper="1.57"
+            effort="0"
+            velocity="0"/>
+    </joint>
+    <link name="left_12">
+        <visual>
+            <origin xyz="0 0 0" rpy="0 0 0"/>
+            <geometry>
+                <mesh filename="package://moria_description/meshes/left_12.STL"/>
+            </geometry>
+            <material name="cyan">
+                <color rgba="0.3137 0.6941 0.7843 1"/>
+            </material>
+        </visual>
+        <collision>
+            <origin xyz="0 0 0" rpy="0 0 0"/>
+            <geometry>
+                <mesh filename="package://moria_description/meshes/left_12.STL"/>
+            </geometry>
+        </collision>
+        <inertial>
+            <origin xyz="0 0 0" rpy="0 0 0"/>
+            <mass value="0.002"/>
+            <inertia
+                ixx="4E-08" ixy="0.0" ixz="0.0"
+                iyy="3E-08" iyz="0.0"
+                izz="4E-08" />
+        </inertial>
+    </link>
+    <!--LEFT MIDDLE-->
+    <joint name="left_20_joint" type="revolute">
+        <parent link="left_lower_arm"/>
+        <child link="left_20"/>
+        <origin xyz="0.0071 0.0060 0.2457" rpy="-1.5708 0 -0.7626"/>
+        <axis xyz="0 0 -1"/>
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
File: moria_description/urdf/moria.urdf.xacro (robot description, xacro)
@@ -388,3 +388,4 @@
     <xacro:include filename="sensors.xacro"/>
     <xacro:include filename="right_arm.xacro"/>
+    <xacro:include filename="left_arm.xacro"/>
 </robot>

File: moria_description/urdf/sensors.xacro (robot description, xacro)
@@ -63,3 +63,16 @@
         </inertial>
     </link>
+    <!-- CAMERA RGB FRAME-->
+    <joint name="camera_rgb_joint" type="fixed">
+        <parent link="camera"/>
+        <child link="camera_rgb_frame"/>
+        <origin xyz="0 0.02 0.015" rpy="0 0 0"/>
+    </joint>
+    <link name="camera_rgb_frame"/>
+    <joint name="camera_depth_joint" type="fixed">
+        <parent link="camera"/>
+        <child link="camera_depth_frame"/>
+        <origin xyz="0 -0.02 0.015" rpy="0 0 0"/>
+    </joint>
+    <link name="camera_depth_frame"/>
 </robot>
