Commit message: modified:   README.md 	modified:   TODOs.todo 	modified:   moria_bringup/package.xml 	modified:   moria_cartographer/CMakeLists.txt 	new file:   moria_cartographer/README.md 	modified:   moria_cartographer/launch/moria_cartograph.launch.py 	new file:   moria_cartographer/launch/moria_vslam.launch.py 	new file:   moria_cartographer/launch/moria_vslam_scan.launch.py 	new file:   moria_cartographer/launch/vslam.launch.py 	modified:   moria_cartographer/package.xml 	new file:   moria_cartographer/run/frontier_exploration.py 	new file:   moria_cartographer/run/map_clear2.py 	new file:   moria_cartographer/run/map_clear3.py 	renamed:    moria_cartographer/launch/wall_track.py -> moria_cartographer/run/wall_track.py 	modified:   moria_cartographer/rviz/moria_slam.rviz 	modified:   moria_description/package.xml 	modified:   moria_description/rviz/model.rviz 	new file:   moria_description/urdf/fixed_left_arm.xacro 	new file:   moria_description/urdf/fixed_right_arm.xacro 	modified:   moria_description/urdf/left_arm.xacro 	modified:   moria_description/urdf/moria.urdf.xacro 	modified:   moria_description/urdf/right_arm.xacro 	modified:   moria_description/urdf/sensors.xacro 	modified:   moria_gazebo/config/my_controllers.yaml 	new file:   moria_gazebo/config/robot_controller.yaml 	modified:   moria_gazebo/joint_names.txt 	modified:   moria_gazebo/launch/btu.launch.py 	modified:   moria_gazebo/launch/btu_big.launch.py 	modified:   moria_gazebo/launch/empty_world.launch.py 	modified:   moria_gazebo/launch/spawn_moria.launch.py 	modified:   moria_gazebo/models/moria/model.sdf 	modified:   moria_gazebo/models/moria/model.urdf 	modified:   moria_gazebo/package.xml

File: moria_description/urdf/left_arm.xacro (robot description, xacro)
@@ -2,9 +2,14 @@
 <robot xmlns:xacro="http://www.ros.org/wiki/xacro">
     <!-- LEFT ARM-->
-    <joint name="left_shoulder_rad_joint" type="continuous">
+    <joint name="left_shoulder_rad_joint" type="revolute">
         <parent link="body"/>
         <child link="left_shoulder_rad"/>
         <origin xyz="0 0.1564 0.505" rpy="1.5708 0 -3.1416"/>
         <axis xyz="0 0 -1"/>
+        <limit
+            lower="0"
+            upper="2.5"
+            effort="3.7"
+            velocity="0.22"/>
     </joint>
     <link name="left_shoulder_rad">
@@ -27,5 +32,5 @@
         <inertial>
             <origin xyz="0 0 0" rpy="0 0 0"/>
-            <mass value="0.1109"/>
+            <mass value="0.224"/>
             <inertia
                 ixx="0.00007" ixy="0.0" ixz="0.0"
@@ -42,6 +47,6 @@
             lower="0"
             upper="2.5"
-            effort="0"
-            velocity="0"/>
+            effort="3.7"
+            velocity="0.22"/>
     </joint>
     <link name="left_shoulder">
@@ -63,5 +68,5 @@
         <inertial>
             <origin xyz="0 0 0" rpy="0 0 0"/>
-            <mass value="0.1576"/>
+            <mass value="0.223"/>
             <inertia
                 ixx="0.00010" ixy="0.0" ixz="0.0"
@@ -71,9 +76,14 @@
     </link>
     <!-- UPPER ARM-->
-    <joint name="left_upper_arm_joint" type="continuous">
+    <joint name="left_upper_arm_joint" type="revolute">
         <parent link="left_shoulder"/>
         <child link="left_upper_arm"/>
         <origin xyz="0 0.0875 -0.0255" rpy="-1.5708 3.14 0"/>
         <axis xyz="0 0 -1"/>
+        <limit
+            lower="0"
+            upper="2.5"
+            effort="6"
+            velocity="0.11"/>
     </joint>
     <link name="left_upper_arm">
@@ -95,5 +105,5 @@
         <inertial>
             <origin xyz="0 0 0" rpy="0 0 0"/>
-            <mass value="0.1608"/>
+            <mass value="0.209"/>
             <inertia
                 ixx="0.00021" ixy="0.0" ixz="0.0"
@@ -111,6 +121,6 @@
             lower="0"
             upper="1.5"
-            effort="0"
-            velocity="0"/>
+            effort="6"
+            velocity="0.11"/>
     </joint>
     <link name="left_elbow">
@@ -132,5 +142,5 @@
         <inertial>
             <origin xyz="0 0 0" rpy="0 0 0"/>
-            <mass value="0.1267"/>
+            <mass value="0.176"/>
             <inertia
                 ixx="0.00010" ixy="0.0" ixz="0.0"
@@ -140,9 +150,14 @@
     </link>
     <!-- LEFT LOWER ARM-->
-    <joint name="left_lower_arm_joint" type="continuous">
+    <joint name="left_lower_arm_joint" type="revolute">
         <parent link="left_elbow"/>
         <child link="left_lower_arm"/>
         <origin xyz="0 0.0866 -0.0234" rpy="-1.5708 2.62 0"/>
         <axis xyz="0 0 -1"/>
+        <limit
+            lower="0"
+            upper="2.5"
+            effort="6"
+            velocity="0.11"/>
     </joint>
     <link name="left_lower_arm">
@@ -164,5 +179,5 @@
         <inertial>
             <origin xyz="0 0 0" rpy="0 0 0"/>
-            <mass value="0.3515"/>
+            <mass value="0.882"/>
             <inertia
                 ixx="0.00033" ixy="0.0" ixz="0.0"

File: moria_description/urdf/moria.urdf.xacro (robot description, xacro)
@@ -306,14 +306,14 @@
     </link>
     <!-- HEAD-->
-    <joint name="neck_joint" type="revolute">
+    <joint name="neck_joint" type="fixed"> <!-- rev-->
         <parent link="body"/>
         <child link="neck"/>
         <origin xyz="0.0092 0.0004 0.5471" rpy="0 0 1.5708"/>
-        <axis xyz="0 0 1"/>
+        <!--<axis xyz="0 0 1"/>
         <limit
             lower="-0.5"
             upper="0.5"
             effort="0"
-            velocity="0"/>
+            velocity="0"/>-->
     </joint>
     <link name="neck">
@@ -342,14 +342,14 @@
         </inertial>
     </link>
-    <joint name="head_joint" type="revolute">
+    <joint name="head_joint" type="fixed"> <!-- rev-->
         <parent link="neck"/>
         <child link="head"/>
         <origin xyz="0.0224 0.004 0.0403" rpy="1.5708 0 1.5708"/>
-        <axis xyz="0 0 1"/>
+        <!--<axis xyz="0 0 1"/>
         <limit
             lower="-0.2"
             upper="0.2"
             effort="0"
-            velocity="0"/>
+            velocity="0"/> -->
     </joint>
     <link name="head">
@@ -379,4 +379,6 @@
     </link>
     <xacro:include filename="sensors.xacro"/>
+    <!-- <xacro:include filename="fixed_right_arm.xacro"/>
+    <xacro:include filename="fixed_left_arm.xacro"/> -->
     <xacro:include filename="right_arm.xacro"/>
     <xacro:include filename="left_arm.xacro"/>

File: moria_description/urdf/right_arm.xacro (robot description, xacro)
@@ -2,9 +2,14 @@
 <robot xmlns:xacro="http://www.ros.org/wiki/xacro">
     <!-- RIGHT ARM-->
-    <joint name="right_shoulder_rad_joint" type="continuous">
+    <joint name="right_shoulder_rad_joint" type="revolute">
         <parent link="body"/>
         <child link="right_shoulder_rad"/>
         <origin xyz="0 -0.1556 0.505" rpy="-1.5708 0 3.1416"/>
         <axis xyz="0 0 1"/>
+        <limit
+            lower="0"
+            upper="2.5"
+            effort="3.7"
+            velocity="0.22"/>
     </joint>
     <link name="right_shoulder_rad">
@@ -27,5 +32,5 @@
         <inertial>
             <origin xyz="0 0 0" rpy="0 0 0"/>
-            <mass value="0.1128"/>
+            <mass value="0.224"/>
             <inertia
                 ixx="0.00007" ixy="0.0" ixz="0.0"
@@ -42,6 +47,6 @@
             lower="0"
             upper="2.5"
-            effort="0"
-            velocity="0"/>
+            effort="3.7"
+            velocity="0.22"/>
     </joint>
     <link name="right_shoulder">
@@ -63,5 +68,5 @@
         <inertial>
             <origin xyz="0 0 0" rpy="0 0 0"/>
-            <mass value="0.1576"/>
+            <mass value="0.223"/>
             <inertia
                 ixx="0.00010" ixy="0.0" ixz="0.0"
@@ -71,9 +76,14 @@
     </link>
     <!-- UPPER ARM-->
-    <joint name="right_upper_arm_joint" type="continuous">
+    <joint name="right_upper_arm_joint" type="revolute">
         <parent link="right_shoulder"/>
         <child link="right_upper_arm"/>
         <origin xyz="0 0.0875 -0.0255" rpy="-1.5708 0 0"/>
         <axis xyz="0 0 1"/>
+        <limit
+            lower="0"
+            upper="2.5"
+            effort="6"
+            velocity="0.11"/>
     </joint>
     <link name="right_upper_arm">
@@ -95,5 +105,5 @@
         <inertial>
             <origin xyz="0 0 0" rpy="0 0 0"/>
-            <mass value="0.1608"/>
+            <mass value="0.209"/>
             <inertia
                 ixx="0.00021" ixy="0.0" ixz="0.0"
@@ -110,7 +120,7 @@
         <limit
             lower="0"
-            upper="1.5"
-            effort="0"
-            velocity="0"/>
+            upper="2.5"
+            effort="6"
+            velocity="0.11"/>
     </joint>
     <link name="right_elbow">
@@ -132,5 +142,5 @@
         <inertial>
             <origin xyz="0 0 0" rpy="0 0 0"/>
-            <mass value="0.1267"/>
+            <mass value="0.176"/>
             <inertia
                 ixx="0.00010" ixy="0.0" ixz="0.0"
@@ -140,9 +150,14 @@
     </link>
     <!-- RIGHT LOWER ARM-->
-    <joint name="right_lower_arm_joint" type="continuous">
+    <joint name="right_lower_arm_joint" type="revolute">
         <parent link="right_elbow"/>
         <child link="right_lower_arm"/>
         <origin xyz="0 0.0866 -0.0222" rpy="-1.5708 1.5708 0"/>
         <axis xyz="0 0 1"/>
+        <limit
+            lower="0"
+            upper="2.5"
+            effort="6"
+            velocity="0.11"/>
     </joint>
     <link name="right_lower_arm">
@@ -164,5 +179,5 @@
         <inertial>
             <origin xyz="0 0 0" rpy="0 0 0"/>
-            <mass value="0.3515"/>
+            <mass value="0.882"/>
             <inertia
                 ixx="0.00033" ixy="0.0" ixz="0.0"

File: moria_description/urdf/sensors.xacro (robot description, xacro)
@@ -73,6 +73,12 @@
         <parent link="camera"/>
         <child link="camera_depth_frame"/>
-        <origin xyz="0 -0.02 0.015" rpy="0 0 0"/>
+        <origin xyz="0 -0.02 0.015" rpy="-1.57 0 -1.57"/>
     </joint>
     <link name="camera_depth_frame"/>
+    <joint name="camera_point_joint" type="fixed">
+        <parent link="camera"/>
+        <child link="camera_point_frame"/>
+        <origin rpy="-1.57 1.57 3.14" xyz="0 0.02 0.015"/>
+    </joint>
+    <link name="camera_point_frame"/>
 </robot>

File: moria_gazebo/models/moria/model.urdf (robot description, URDF)
Before this commit: robot moria, 56 links, 55 joints
Links:
- added link camera_point_frame
- link base_link: geometry collision mesh filename=model://moria/meshes/base_link.STL; visual mesh filename=model://moria/meshes/base_link.STL
- link body: geometry collision mesh filename=model://moria/meshes/body.STL; visual mesh filename=model://moria/meshes/body.STL
- link camera: geometry collision mesh filename=model://moria/meshes/camera.STL; visual mesh filename=model://moria/meshes/camera.STL
- link front_base: geometry collision mesh filename=model://moria/meshes/front_base.STL; visual mesh filename=model://moria/meshes/front_base.STL
- link front_radial: geometry collision mesh filename=model://moria/meshes/front_rad.STL; visual mesh filename=model://moria/meshes/front_rad.STL
- link front_wheel: geometry collision mesh filename=model://moria/meshes/front_wheel.STL; visual mesh filename=model://moria/meshes/front_wheel.STL
- link head: geometry collision mesh filename=model://moria/meshes/head.STL; visual mesh filename=model://moria/meshes/head.STL
- link left_00: geometry collision mesh filename=model://moria/meshes/left_00.STL; visual mesh filename=model://moria/meshes/left_00.STL
- link left_01: geometry collision mesh filename=model://moria/meshes/left_01.STL; visual mesh filename=model://moria/meshes/left_01.STL
- link left_02: geometry collision mesh filename=model://moria/meshes/left_02.STL; visual mesh filename=model://moria/meshes/left_02.STL
- link left_10: geometry collision mesh filename=model://moria/meshes/left_10.STL; visual mesh filename=model://moria/meshes/left_10.STL
- link left_11: geometry collision mesh filename=model://moria/meshes/left_11.STL; visual mesh filename=model://moria/meshes/left_11.STL
- link left_12: geometry collision mesh filename=model://moria/meshes/left_12.STL; visual mesh filename=model://moria/meshes/left_12.STL
- link left_20: geometry collision mesh filename=model://moria/meshes/left_20.STL; visual mesh filename=model://moria/meshes/left_20.STL
- link left_21: geometry collision mesh filename=model://moria/meshes/left_21.STL; visual mesh filename=model://moria/meshes/left_21.STL
- link left_22: geometry collision mesh filename=model://moria/meshes/left_22.STL; visual mesh filename=model://moria/meshes/left_22.STL
- link left_30: geometry collision mesh filename=model://moria/meshes/left_30.STL; visual mesh filename=model://moria/meshes/left_30.STL
- link left_31: geometry collision mesh filename=model://moria/meshes/left_31.STL; visual mesh filename=model://moria/meshes/left_31.STL
- link left_32: geometry collision mesh filename=model://moria/meshes/left_32.STL; visual mesh filename=model://moria/meshes/left_32.STL
- link left_40: geometry collision mesh filename=model://moria/meshes/left_40.STL; visual mesh filename=model://moria/meshes/left_40.STL
- link left_41: geometry collision mesh filename=model://moria/meshes/left_41.STL; visual mesh filename=model://moria/meshes/left_41.STL
- link left_42: geometry collision mesh filename=model://moria/meshes/left_42.STL; visual mesh filename=model://moria/meshes/left_42.STL
- link left_elbow: mass 0.1267 -> 0.176; geometry collision mesh filename=model://moria/meshes/left_elbow.STL; visual mesh filename=model://moria/meshes/left_elbow.STL
- link left_lower_arm: mass 0.3515 -> 0.882; geometry collision mesh filename=model://moria/meshes/left_lower_arm.STL; visual mesh filename=model://moria/meshes/left_lower_arm.STL
- link left_motor: geometry collision mesh filename=model://moria/meshes/left_motor.STL; visual mesh filename=model://moria/meshes/left_motor.STL
- link left_shoulder: mass 0.1576 -> 0.223; geometry collision mesh filename=model://moria/meshes/left_shoulder.STL; visual mesh filename=model://moria/meshes/left_shoulder.STL
- link left_shoulder_rad: mass 0.1109 -> 0.224; geometry collision mesh filename=model://moria/meshes/left_shoulder_rad.STL; visual mesh filename=model://moria/meshes/left_shoulder_rad.STL
- link left_upper_arm: mass 0.1608 -> 0.209; geometry collision mesh filename=model://moria/meshes/left_upper_arm.STL; visual mesh filename=model://moria/meshes/left_upper_arm.STL
- link left_wheel: geometry collision mesh filename=model://moria/meshes/left_wheel.STL; visual mesh filename=model://moria/meshes/left_wheel.STL
- link leg: geometry collision mesh filename=model://moria/meshes/leg.STL; visual mesh filename=model://moria/meshes/leg.STL
- link lidar: geometry collision mesh filename=model://moria/meshes/lidar.STL; visual mesh filename=model://moria/meshes/lidar.STL
- link neck: geometry collision mesh filename=model://moria/meshes/neck.STL; visual mesh filename=model://moria/meshes/neck.STL
- link right_00: geometry collision mesh filename=model://moria/meshes/right_00.STL; visual mesh filename=model://moria/meshes/right_00.STL
- link right_01: geometry collision mesh filename=model://moria/meshes/right_01.STL; visual mesh filename=model://moria/meshes/right_01.STL
- link right_02: geometry collision mesh filename=model://moria/meshes/right_02.STL; visual mesh filename=model://moria/meshes/right_02.STL
- link right_10: geometry collision mesh filename=model://moria/meshes/right_10.STL; visual mesh filename=model://moria/meshes/right_10.STL
- link right_11: geometry collision mesh filename=model://moria/meshes/right_11.STL; visual mesh filename=model://moria/meshes/right_11.STL
- link right_12: geometry collision mesh filename=model://moria/meshes/right_12.STL; visual mesh filename=model://moria/meshes/right_12.STL
- link right_20: geometry collision mesh filename=model://moria/meshes/right_20.STL; visual mesh filename=model://moria/meshes/right_20.STL
- link right_21: geometry collision mesh filename=model://moria/meshes/right_21.STL; visual mesh filename=model://moria/meshes/right_21.STL
- link right_22: geometry collision mesh filename=model://moria/meshes/right_22.STL; visual mesh filename=model://moria/meshes/right_22.STL
- link right_30: geometry collision mesh filename=model://moria/meshes/right_30.STL; visual mesh filename=model://moria/meshes/right_30.STL
- link right_31: geometry collision mesh filename=model://moria/meshes/right_31.STL; visual mesh filename=model://moria/meshes/right_31.STL
- link right_32: geometry collision mesh filename=model://moria/meshes/right_32.STL; visual mesh filename=model://moria/meshes/right_32.STL
- link right_40: geometry collision mesh filename=model://moria/meshes/right_40.STL; visual mesh filename=model://moria/meshes/right_40.STL
- link right_41: geometry collision mesh filename=model://moria/meshes/right_41.STL; visual mesh filename=model://moria/meshes/right_41.STL
- link right_42: geometry collision mesh filename=model://moria/meshes/right_42.STL; visual mesh filename=model://moria/meshes/right_42.STL
- link right_elbow: mass 0.1267 -> 0.176; geometry collision mesh filename=model://moria/meshes/right_elbow.STL; visual mesh filename=model://moria/meshes/right_elbow.STL
- link right_lower_arm: mass 0.3515 -> 0.882; geometry collision mesh filename=model://moria/meshes/right_lower_arm.STL; visual mesh filename=model://moria/meshes/right_lower_arm.STL
- link right_motor: geometry collision mesh filename=model://moria/meshes/right_motor.STL; visual mesh filename=model://moria/meshes/right_motor.STL
- link right_shoulder: mass 0.1576 -> 0.223; geometry collision mesh filename=model://moria/meshes/right_shoulder.STL; visual mesh filename=model://moria/meshes/right_shoulder.STL
- link right_shoulder_rad: mass 0.1128 -> 0.224; geometry collision mesh filename=model://moria/meshes/right_shoulder_rad.STL; visual mesh filename=model://moria/meshes/right_shoulder_rad.STL
- link right_upper_arm: mass 0.1608 -> 0.209; geometry collision mesh filename=model://moria/meshes/right_upper_arm.STL; visual mesh filename=model://moria/meshes/right_upper_arm.STL
- link right_wheel: geometry collision mesh filename=model://moria/meshes/right_wheel.STL; visual mesh filename=model://moria/meshes/right_wheel.STL
Joints:
- added joint camera_point_joint: type fixed, parent camera, child camera_point_frame, origin xyz=0 0.02 0.015 rpy=1.57 3.14 0
- joint left_elbow_joint: limit lower=0 upper=1.5 effort=10 velocity=2 -> lower=0 upper=2.5 effort=6 velocity=0.11
- joint left_lower_arm_joint: limit (none) -> lower=0 upper=2.5 effort=6 velocity=0.11; type continuous -> revolute
- joint left_shoulder_joint: limit lower=0 upper=2.5 effort=10 velocity=2 -> lower=0 upper=2.5 effort=3.7 velocity=0.22
- joint left_shoulder_rad_joint: axis 0 0 -1 -> (none); type continuous -> fixed
- joint left_upper_arm_joint: limit (none) -> lower=0 upper=2.5 effort=6 velocity=0.11; type continuous -> revolute
- joint right_elbow_joint: limit lower=0 upper=1.5 effort=10 velocity=2 -> lower=0 upper=2.5 effort=6 velocity=0.11
- joint right_lower_arm_joint: limit (none) -> lower=0 upper=2.5 effort=6 velocity=0.11; type continuous -> fixed
- joint right_shoulder_joint: limit lower=0 upper=2.5 effort=10 velocity=2 -> lower=0 upper=2.5 effort=3.7 velocity=0.22
- joint right_shoulder_rad_joint: limit (none) -> lower=0 upper=2.5 effort=3.7 velocity=0.22; type continuous -> revolute
- joint right_upper_arm_joint: limit (none) -> lower=0 upper=2.5 effort=6 velocity=0.11; type continuous -> revolute
